File: Hardware/STM32C071.kicad_pcb (KiCad board)
At the start: 2 copper layers, 50 x 25 mm, 15 parts, among them J1 USB_C_Receptacle_USB2.0_16P, U1 STM32C071K8Tx, U2 USBLC6-2P6, U4 XL1509-ADJE1

Commit message: Added SWD connector and 3D view
Parts:
- added J2: Conn_01x04_Pin, Connector_PinHeader_2.54mm:PinHeader_1x04_P2.54mm_Horizontal, F.Cu at (123.1, 90.0)
- moved U1 8.40 mm to (132.2, 88.5)
Connections:
- J1 pad 0: GND -> (no net)
- U1 pad 24: unconnected-(U1-PA13-Pad24) -> Net-(J2-Pin_3)
- U1 pad 25: unconnected-(U1-PA14-Pad25) -> Net-(J2-Pin_2)
- U2 pad 1: Net-(U1-PA11) -> Net-(U1-PA12)
- U2 pad 3: Net-(U1-PA12) -> Net-(U1-PA11)
- U2 pad 4: Net-(J1-D+-PadA6) -> Net-(J1-D--PadA7)
- U2 pad 6: Net-(J1-D--PadA7) -> Net-(J1-D+-PadA6)
Routing:
- net Net-(U1-PA12): track 0.00 -> 18.8 mm
- net Net-(U1-PA11): track 0.00 -> 18.5 mm
- net +3.3V: track 11.4 -> 27.5 mm, vias 0 -> 1
- net Net-(J2-Pin_3): track 0.00 -> 11.6 mm
- net Net-(J2-Pin_2): track 0.00 -> 10.3 mm
- net GND: track 35.1 -> 36.0 mm, vias 9 -> 10
